Commit message: Update mybot.urdf

File: src/bot_model/urdf/mybot.urdf (robot description, URDF)
Before this commit: robot mybot, 4 links, 3 joints
Joints:
- joint base_front: limit lower=-0.7 upper=0.7 effort=1 velocity=3 -> lower=-0.7 upper= 0.7  effort= 1   velocity= 3  

Commit message: added diff drive plugin

File: src/bot_model/urdf/mybot.urdf (robot description, URDF)
Before this commit: robot mybot, 4 links, 3 joints
Joints:
- joint base_left_rear_wheel: limit lower=-0.7 upper=0.7 effort=1 velocity=3 -> effort=1 velocity=3; type revolute -> continuous
- joint base_right_rear_wheel: limit lower=-0.7 upper=0.7 effort=1 velocity=3 -> effort=1 velocity=3; type revolute -> continuous

Commit message: changed the model and added diff drive plugin

File: src/bot_model/urdf/mybot.urdf (robot description, URDF)
Before this commit: robot mybot, 4 links, 3 joints
Links:
- removed link base
- removed link front_wheel
- removed link left_rear_wheel
- removed link right_rear_wheel
- added link base_footprint; visual box size=0.001 0.001 0.001
- added link base_link, mass 1; collision box size=0.16 0.106 0.01; visual box size=0.16 0.106 0.01
- added link caster_wheel, mass 0.5; collision sphere radius=0.0175; visual sphere radius=0.0175
- added link left_wheel, mass 1; collision cylinder length=0.005 radius=0.035; visual cylinder length=0.005 radius=0.035
- added link right_wheel, mass 1; collision cylinder length=0.005 radius=0.035; visual cylinder length=0.005 radius=0.035
Joints:
- removed joint base_front
- removed joint base_left_rear_wheel
- removed joint base_right_rear_wheel
- added joint base_link_joint: type fixed, parent base_footprint, child base_link, origin xyz=0 0 0.04 rpy=0 0 0
- added joint caster_wheel_joint: type continuous, parent base_link, child caster_wheel, origin xyz=-0.052 0 -0.0225 rpy=0 0 0, axis 0 1 0
- added joint left_wheel_joint: type continuous, parent base_link, child left_wheel, origin xyz=0.02 0.06 -0.005 rpy=0 0 0, axis 0 1 0
- added joint right_wheel_joint: type continuous, parent base_link, child right_wheel, origin xyz=0.02 -0.06 -0.005 rpy=0 0 0, axis 0 1 0

Commit message: added stereo cam plugin

File: src/bot_model/urdf/mybot.urdf (robot description, URDF)
Before this commit: robot mybot, 5 links, 4 joints
Links:
- added link camera_link, mass 1e-5; collision box size=0.01 0.01 0.01; visual box size=0.01 0.01 0.01
Joints:
- added joint camera_joint: type fixed, parent base_link, child camera_link, origin xyz=0.03 0 0.04  rpy=0 0 0, axis 0 1 0
